Commit message: Update lidar.xacro

File: description/lidar.xacro (robot description, xacro)
@@ -0,0 +1,10 @@
+<?xml version="1.0"?>
+<robot xmlns:xacro="http://www.ros.org/wiki/xacro"  name="robot">
+  <joint name="lidar_joint" type="fixed">
+    <parent link="chassis" />
+    <child link="lidar_frame" />
+    <origin xyz="0.1 0 0.175" rpy="0 0 0" />
+  </joint>
+  <link name="lidar_frame">
+  </link>
+</robot>

Commit message: Update lidar.xacro

File: description/lidar.xacro (robot description, xacro)
@@ -7,4 +7,18 @@
   </joint>
   <link name="lidar_frame">
+     <visual>
+      <geometry>
+          <cylinder radius="0.05" length="0.04"/>
+        </geometry>
+        <material name="white" />
+      </visual>
+      <collision>
+        <geometry>
+          <cylinder radius="0.05" length="0.04"/>
+        </geometry>
+      </collision>
+      <xacro:inertial_cylinder mass="0.1" length="0.04" radius="0.05">
+        <origin xyz="0 0 0" rpy="0 0 0"/>
+      </xacro:inertial_cylinder>
   </link>
 </robot>

Commit message: Update lidar.xacro

File: description/lidar.xacro (robot description, xacro)
@@ -22,3 +22,31 @@
       </xacro:inertial_cylinder>
   </link>
+  <gazebo reference="lidar_frame">
+        <material>Gazebo/Red</material>
+        <sensor name="laser" type="ray">
+            <pose> 0 0 0 0 0 0 </pose>
+            <visualize>true</visualize>
+            <update_rate>10</update_rate>
+            <ray>
+                <scan>
+                    <horizontal>
+                        <samples>360</samples>
+                        <min_angle>-3.14</min_angle>
+                        <max_angle>3.14</max_angle>
+                    </horizontal>
+                </scan>
+                <range>
+                    <min>0.3</min>
+                    <max>12</max>
+                </range>
+            </ray>
+            <plugin name="laser_controller" filename="libgazebo_ros_ray_sensor.so">
+                <ros>
+                    <argument>~/out:=scan</argument>
+                </ros>
+                <output_type>sensor_msgs/LaserScan</output_type>
+                <frame_name>lidar_frame</frame_name>
+            </plugin>
+        </sensor>
+  </gazebo>
 </robot>
